File: Eagle/Balloon_Cut-Down.sch (EAGLE design)
At the start: 64 parts, among them Q1 DMG3415U-7, U1 MCP111T-240E/TT, U2 SPX3819-3.3, U3 MPM3610, U4 74AHCT1G125DBV, U5 ATSAMD21G18_QFN, X1 32.768

Commit message: Major update for the V3 PCB
Major update for the V3 PCB: the cut-down is now based on the eRIC4 or eRIC9 radio controller and can be triggered by radio; a u-blox CAM-M8Q provides altitude information; the Shark and Servo are now mounted directly on the PCB instead of carbon fibre. The V1 files are in the Archive folder.
Parts:
- removed !RST, 3V3, 3V3SW1, 3V3SW2, CLOSE, GND3, GND4, GND5, OPEN, RX, SCL, SDA, SWCLK, SWDIO, TX, VBUS: (no value), adafruit:PINHD-1X1
- removed C12: 0.1uF, microbuilder:CAP_CERAMIC0805-NOOUTLINE
- removed C13, C14, C15, C16: 10nF, rcl:C-EUC0805
- removed CON1: (no value), microbuilder:USBFCI_10103594
- removed LED: RED, adafruit:LED3MM
- removed S5: SWITCH-MOMENTARY-2PTH, SparkFun-Electromechanical:SWITCH-MOMENTARY-2PTH
- removed U1: MCP111T-240E/TT, Microchip-MCP11:MCP111T-270E/TT
- removed U2: SPX3819-3.3, microbuilder:VREG_SOT23-5
- removed U3: MPM3610, IntegratedCircuits:2093_MPM3610GQV-P
- removed U4: 74AHCT1G125DBV, 74xx-little-us:74AHCT1G125DBV
- removed U5: ATSAMD21G18_QFN, microbuilder:ATSAMD21J_QFN
- added BOOT1, BOOT2, CTS, RTS, RXD, TXD, VCC: (no value), adafruit:PINHD-1X1
- added D3: MBR120, microbuilder:DIODE-SCHOTTKYSOD-123
- added FREQ: (no value), microbuilder:SOLDERJUMPER
- added IC1: ERIC9-FCC, SamacSys_Parts:ERIC9-FCC
- added IC2: MCP111T-240E/TT, Microchip-MCP11:MCP111T-270E/TT
- added IC3: CAM-M8, ubloxLib:CAM-M8
- added IC4: SPX3819-3.3, microbuilder:VREG_SOT23-5
- added IC5: MPM3610, IntegratedCircuits:2093_MPM3610GQV-P
- added IC6: 74AHCT1G125DBV, 74xx-little-us:74AHCT1G125DBV
- added LED1: RED, microbuilder:LED0805_NOOUTLINE
- added RESET: SWITCH-MOMENTARY-2PTH, SparkFun-Electromechanical:SWITCH-MOMENTARY-2PTH
- BAT: device SparkFun-Electromechanical:BATTERYBATTERY-9V-KEYSTONE1294 -> SparkFun-Electromechanical:BATTERYBATTERY-9V-KEYSTONE-593-594
- C1: value 1uF -> 10µF; device microbuilder:CAP_CERAMIC0603_NO -> microbuilder:CAP_CERAMIC0805-NOOUTLINE
- C10: value 22uF -> 1nF
- C2: value 12pF -> 10µF; device microbuilder:CAP_CERAMIC0603_NO -> microbuilder:CAP_CERAMIC0805-NOOUTLINE
- C3: value 12pF -> 100nF
- C4: value 10µF -> 10uF; device microbuilder:CAP_CERAMIC0805-NOOUTLINE -> rcl:C-EUC0805
- C5: device microbuilder:CAP_CERAMIC0805-NOOUTLINE -> rcl:C-EUC0805
- C6: value 10µF -> 10nF; device microbuilder:CAP_CERAMIC0805-NOOUTLINE -> rcl:C-EUC0805
- C7: value 10nF -> 0.1uF; device rcl:C-EUC0805 -> microbuilder:CAP_CERAMIC0805-NOOUTLINE
- C8: value 1uF -> 10nF; device microbuilder:CAP_CERAMIC0603_NO -> rcl:C-EUC0805
- C9: value 10uF -> 10nF
- R1, R7, R8: value 2.2K -> 1K
- X1: value 32.768 -> BU-SMA-V; device adafruit2:XTAL-3.2X1.5 -> con-coax:BU-SMA-V
Connections:
- removed net A0: C15.2, S4.2, U5.PA02/EINT2/AIN0/Y0/VOUT
- removed net A1: C13.2, OPEN.1, S2.2, U5.PB08/I8/AIN2/SERCOM4.0
- removed net A2: C14.2, CLOSE.1, S3.2, U5.PB09/I9/AIN3/SERCOM4.1
- removed net A3: U5.PA04/EINT4/VREFB/AIN4/SERCOM0.0
- removed net A4: U5.PA05/EINT5/AIN5/SERCOM0.1
- removed net A5: C16.2, S5.2, U5.PB02/I2/AIN10/SERCOM5.0
- removed net AREF: C8.1, U5.PA03/EINT3/VREFA/AIN1
- removed net D+: CON1.D+, U5.PA25/I13/SERCOM3+5.3/D+
- removed net D-: CON1.D-, U5.PA24/I12/SERCOM3+5.2/D-
- removed net D0: RX.1, U5.PA11/I11/AIN19/SERCOM0+2.3/I2SF0
- removed net D1: TX.1, U5.PA10/I10/AIN18/SERCOM0+2.2/I2SCK
- removed net D10: U5.PA18/I2/SERCOM1+3.2
- removed net D11: Q1.G, R9.2, U5.PA16/I2C/I0/SERCOM1+3.0
- removed net D12: U5.PA19/I3/SERCOM1+3.3/I2SD0
- removed net D13: R1.1, U5.PA17/I2C/I1/SERCOM1+3.1
- removed net D2: U5.PA14/I14/SERCOM2+4.2
- removed net D3: U5.PA09/I2C/I9/AIN17/SERCOM0+2.1/I2SMC
- removed net D5: U4A.I, U5.PA15/I15/SERCOM3+4.3
- removed net D6: U5.PA20/I4/SERCOM3+5.2/I2SSC
- removed net D7: U5.PA21/I5/SERCOM3+5.3/I2SFS0
- removed net D8: U3.EN, U5.PA06/EINT6/AIN6/SERCOM0.2
- removed net D9: R2.1, R3.2, U5.PA07/I7/AIN7/SERCOM0.3/I2SD0
- removed net MISO: U5.PA12/I12/I2C/SERCOM2+4.0
- removed net MOSI: U5.PB10/I10/SERCOM4.2/I2SMC
- removed net N$16: CON1.VBUS, D2.A
- removed net N$5: C2.1, U5.PA00/EINT0/SERCOM1.0, X1.P$1
- removed net N$7: C3.1, U5.PA01/EINT1/SERCOM1.1, X1.P$2
- removed net SCK: U5.PB11/I11/SERCOM4.3/I2SCL
- removed net SCL: R7.2, SCL.1, U5.PA23/I2C/I7/SERCOM3+5.1/SOF
- removed net SDA: R8.2, SDA.1, U5.PA22/I2C/I6/SERCOM3+5.0
- removed net SD_CS: U5.PA08/I2C/AIN16/SERCOM0+2.0/I2SD1
- removed net SWCLK: SWCLK.1, U5.PA30/I10/SECOM1.2/SWCLK
- removed net SWDIO: SWDIO.1, U5.PA31/I11/SECOM1.3/SWDIO
- removed net VDDCORE1: C1.1, U5.VDDCORE
- new net CTS: C9.2, CTS.1, IC1.BUSY, S2.2
- new net FREQ: FREQ.1, IC1.INPUT
- new net N$1: R7.1, TXD.1
- new net N$2: IC3.RF_IN, IC3.RF_OUT
- new net N$4: R8.1, RTS.1
- new net N$6: C4.1, D3.C, IC5.VIN
- new net N$9: D2.A, VCC.1
- new net PIN10: IC1.GPIO_1, Q1.G, R9.2
- new net PIN11: BOOT1.1, IC1.GPIO_2
- new net PIN12: BOOT2.1, IC1.GPIO_3
- new net PIN13: IC1.GPIO_4, IC5.EN
- new net PIN15: IC1.GPIO_5, IC3.RXD/SPI_MOSI
- new net PIN16: IC1.GPIO_6, R1.1
- new net PIN17: IC1.GPIO_7, IC3.TXD/SPI_MISO
- new net PIN18: IC1.GPIO_8, IC6A.I
- new net PIN19: IC1.GPIO_9
- new net PIN20: IC1.GPIO_10
- new net PIN21: IC1.GPIO_11
- new net PIN22: IC1.GPIO_12, R2.1, R3.2
- new net RF: IC1.RF, X1.1
- new net RTS: C11.2, IC1.HOST_READY, R8.2, S4.2
- new net RXD: C8.2, IC1.SDO, RXD.1, S1.2
- new net TXD: C10.2, IC1.SDI, R7.2, S3.2
- net !RESET: now also IC1.RESET, IC2.VOUT, IC3.!RESET, RESET.2; no longer !RST.1, S1.1, U1.VOUT, U5./RESET
- net +3V3: now also C2.1, C3.1, IC1.VCC, IC2.VDD, IC3.V_BCKP, IC4.OUT; no longer 3V3.1, C5.1, C6.1, C7.1, R7.1, R8.1, U1.VDD, U2.OUT, U5.VDDA, U5.VDDIN, U5.VDDIO
- net +5V: now also C5.1, C6.1, IC5.OUT, IC6P.VCC; no longer C10.1, C11.1, U3.OUT, U4P.VCC
- net 3V3SW: now also C7.1, IC3.VCC, IC3.VCC_IO; no longer 3V3SW1.1, 3V3SW2.1, C12.1
- net GND: now also C10.1, C11.1, C8.1, C9.1, FREQ.2, IC1.GND, IC1.RF_GND, IC2.VSS, IC3.GND$1, IC3.GND$10, IC3.GND$11, IC3.GND$12, IC3.GND$13, IC3.GND$14, IC3.GND$2, IC3.GND$3, IC3.GND$4, IC3.GND$5, IC3.GND$6, IC3.GND$7, IC3.GND$8, IC3.GND$9, IC4.GND, IC5.AGND, IC5.GND, IC6A.OE, IC6P.GND, LED1.C, RESET.1, S1.1, X1.2; no longer C10.2, C11.2, C12.2, C13.1, C14.1, C15.1, C16.1, C8.2, C9.2, CON1.GND, GND3.1, GND4.1, GND5.1, LED.C, S1.2, S5.1, U1.VSS, U2.GND, U3.AGND, U3.GND, U4A.OE, U4P.GND, U5.GND, U5.GNDA
- net N$26: now also IC5.FB; no longer U3.FB
- net N$29: now also IC5.AAM; no longer U3.AAM
- net N$3: now also LED1.A; no longer LED.A
- net PWM: now also IC6A.O; no longer U4A.O
- net VBAT: now also D3.A; no longer C9.1, U3.VIN
- net VBUS: now also C1.1, IC4.EN, IC4.IN; no longer C4.1, U2.EN, U2.IN, VBUS.1
Other:
- note added: "Balloon Cut-Down Device V3"
- note added: "Energiser Ultimate Lithium 9V in Keystone Electronics 593 and 594 clips"
- note added: "u-blox CAM-M8"
- note removed: "BREAKOUTS"
- note removed: "Balloon Cut-Down Device"
- note removed: "Energiser Ultimate Lithium 9V in Keystone Electronics 1294 clip"
- note removed: "LED"
- note removed: "MICROCONTROLLER"
- note removed: "N/C"
- note removed: "POWER AND FILTERING"
- note removed: "RESET"
- note removed: "RXD"
- note removed: "RXLED"
- note removed: "TXD"
- note removed: "TXLED"
- note removed: "USB"
- note removed: "USBHOSTEN"
- note removed: "With grateful thanks to: Adafruit for the Feather M0 Adalogger https://www.adafruit.com/products/2796 https://github.com/adafruit/Adafruit-Feather-M0-Adalogger-PCB Adafruit invests time and resources providing this open source design, please support Adafruit and open-source hardware by purchasing products from Adafruit! Designed by Adafruit Industries."
